Commit message: 默认坐标系

File: urdf/chyPapa3/urdf/chyPapa3.urdf (robot description, URDF)
Before this commit: robot chyPapa3, 13 links, 12 joints
Joints:
- joint Joint_arm_shoulder_le: axis 0 0 -1 -> -0.18328 -0.0084218 -0.98302; limit lower=-1.5 upper=1.5 effort=0 velocity=0 -> lower=-1.5 upper=1.5 effort=100 velocity=0
- joint Joint_arm_shoulder_lf: limit lower=-1.5 upper=1.5 effort=0 velocity=0 -> lower=-1.5 upper=1.5 effort=100 velocity=0
- joint Joint_arm_shoulder_re: limit lower=-1.5 upper=1.5 effort=0 velocity=0 -> lower=-1.5 upper=1.5 effort=100 velocity=0; origin xyz=-0.0015198 0.0019631 -0.063813 rpy=-1.5493 0.010135 1.6433 -> xyz=-0.0030423 0.052147 0.033994 rpy=-1.5493 0.010135 1.6433
- joint Joint_arm_shoulder_rf: limit lower=-1.5 upper=1.5 effort=0 velocity=0 -> lower=-1.5 upper=1.5 effort=100 velocity=0
- joint Joint_hand_arm_le: axis 0 0 1 -> -0.1261 -0.0059587 -0.992; limit lower=-1.5 upper=1.5 effort=0 velocity=0 -> lower=-1.5 upper=1.5 effort=100 velocity=0; origin xyz=-0.17397 -0.037994 -0.039 rpy=-3.1416 0 1.5708 -> xyz=-0.15397 -0.022994 -0.019171 rpy=-3.1416 0 -3.0485
- joint Joint_hand_arm_lf: limit lower=-1.5 upper=1.5 effort=0 velocity=0 -> lower=-1.5 upper=1.5 effort=100 velocity=0; origin xyz=-0.15 0.015 -0.037 rpy=3.1416 0 1.5708 -> xyz=-0.13 0 -0.034011 rpy=3.1416 0 3.0138
- joint Joint_hand_arm_re: limit lower=-1.5 upper=1.5 effort=0 velocity=0 -> lower=-1.5 upper=1.5 effort=100 velocity=0; origin xyz=-0.15 0.015 -0.037 rpy=3.1416 0 1.5708 -> xyz=-0.13 0 0 rpy=-3.1416 0 -3.0781
- joint Joint_hand_arm_rf: limit lower=-1.5 upper=1.5 effort=0 velocity=0 -> lower=-1.5 upper=1.5 effort=100 velocity=0; origin xyz=-0.18275 0.015568 -0.039 rpy=-3.1416 0 1.5708 -> xyz=-0.16275 0.00056766 -0.032234 rpy=3.1416 0 2.6822
- joint Joint_shoulder_body_le: limit lower=-0.5 upper=1.5 effort=0 velocity=0 -> lower=-0.5 upper=1.5 effort=100 velocity=0
- joint Joint_shoulder_body_lf: axis 1 0 0 -> 0.049886 -0.41855 0.90682; limit lower=-0.5 upper=1.5 effort=0 velocity=0 -> lower=-0.5 upper=1.5 effort=100 velocity=0
- joint Joint_shoulder_body_re: axis 1 0 0 -> 0 0 0; limit lower=-0.5 upper=1.5 effort=0 velocity=0 -> lower=-0.5 upper=1.5 effort=100 velocity=0; origin xyz=-0.265 -0.14754 -0.021932 rpy=1.1323 0.12088 3.0913 -> xyz=-0.31205 -0.21515 -0.11184 rpy=1.1323 0.12088 3.0913
- joint Joint_shoulder_body_rf: axis 1 0 0 -> -0.28602 -0.95822 0; limit lower=-0.5 upper=1.5 effort=0 velocity=0 -> lower=-0.5 upper=1.5 effort=100 velocity=0; type revolute -> continuous
