Commit message: 加坐标系

File: urdf/chyPapa4/urdf/chyPapa4.urdf (robot description, URDF)
Before this commit: robot chyPapa4, 2 links, 1 joints
Joints:
- joint Joint_Shoulder_Body_fl: type continuous -> revolute

Commit message: 最简urdf2

File: urdf/chyPapa4/urdf/chyPapa4.urdf (robot description, URDF)
Before this commit: robot chyPapa4, 2 links, 1 joints
Links:
- link Link_Shoulder_fl: mass 0.100243096491449 -> 0.034142
- link base_link: mass 0.322564149559201 -> 0.042074
Joints:
- joint Joint_Shoulder_Body_fl: axis 0.049886 -0.41855 0.90682 -> 0 0 1; limit lower=-0.5 upper=1.5 effort=100 velocity=0 -> lower=-1.5 upper=1.5 effort=100 velocity=0; origin xyz=-0.03504 -0.30624 0.013326 rpy=1.123 0.29832 3.0894 -> xyz=-0.040882 -0.025286 -0.0003707 rpy=1.5708 0 0

Commit message: link 加座标系

File: urdf/chyPapa4/urdf/chyPapa4.urdf (robot description, URDF)
Before this commit: robot chyPapa4, 2 links, 1 joints
Links:
- link Link_Shoulder_fl: mass 0.034142 -> 0.0341422557519
- link base_link: mass 0.042074 -> 0.0420735853495988
Joints:
- joint Joint_Shoulder_Body_fl: axis 0 0 1 -> -1 0 0; origin xyz=-0.040882 -0.025286 -0.0003707 rpy=1.5708 0 0 -> xyz=-0.040882 -0.025286 -0.0003707 rpy=1.5708 1.5708 0

Commit message: link 座标系

File: urdf/chyPapa4/urdf/chyPapa4.urdf (robot description, URDF)
Before this commit: robot chyPapa4, 2 links, 1 joints
Joints:
- joint Joint_Shoulder_Body_fl: origin xyz=-0.040882 -0.025286 -0.0003707 rpy=1.5708 1.5708 0 -> xyz=0.008 0.01209 -0.052337 rpy=-1.3308 0 0

Commit message: 布局混乱修改

File: urdf/chyPapa4/urdf/chyPapa4.urdf (robot description, URDF)
Before this commit: robot chyPapa4, 2 links, 1 joints
Links:
- link Link_Shoulder_fl: mass 0.0341422557519 -> 0.034142
- link base_link: mass 0.0420735853495988 -> 0.108265195096751
Joints:
- joint Joint_Shoulder_Body_fl: axis -1 0 0 -> 0 0 1; origin xyz=0.008 0.01209 -0.052337 rpy=-1.3308 0 0 -> xyz=-0.030882 -0.035286 0.022629 rpy=0 0 -0.034445

Commit message: DH坐标系

File: urdf/chyPapa4/urdf/chyPapa4.urdf (robot description, URDF)
Before this commit: robot chyPapa4, 2 links, 1 joints
Links:
- link base_link: mass 0.108265195096751 -> 0.10827
Joints:
- joint Joint_Shoulder_Body_fl: origin xyz=-0.030882 -0.035286 0.022629 rpy=0 0 -0.034445 -> xyz=0 0 0 rpy=0 0 0
