Commit message: DH坐标系建机器人

File: urdf/chyPapa5/urdf/chyPapa5.urdf (robot description, URDF)
Before this commit: robot chyPapa5, 2 links, 1 joints
Links:
- removed link Link_Shoulder
- added link Link_Shoulder_le, mass 0.10024; collision mesh filename=package://chyPapa5/meshes/Link_Shoulder_le.STL; visual mesh filename=package://chyPapa5/meshes/Link_Shoulder_le.STL
- link base_link: mass 0.32256 -> 0.30228
Joints:
- removed joint Joint_Shoulder
- added joint Joint_Shoulder_le: type revolute, parent base_link, child Link_Shoulder_le, origin xyz=-0.071696 -0.03752 -0.019059 rpy=-1.5708 1.5707 -1.5489, axis 0 0 1, limit lower=-0.5 upper=1.5 effort=100 velocity=0

Commit message: DHtest1

File: urdf/chyPapa5/urdf/chyPapa5.urdf (robot description, URDF)
Before this commit: robot chyPapa5, 2 links, 1 joints
Links:
- link Link_Shoulder_le: mass 0.10024 -> 0.09716
- link base_link: mass 0.30228 -> 0.302284486397825
Joints:
- joint Joint_Shoulder_le: origin xyz=-0.071696 -0.03752 -0.019059 rpy=-1.5708 1.5707 -1.5489 -> xyz=-0.0725 -0.019059 0.035943 rpy=-1.5708 -0.00010338 -1.5708

Commit message: DH坐标系2

File: urdf/chyPapa5/urdf/chyPapa5.urdf (robot description, URDF)
Before this commit: robot chyPapa5, 2 links, 1 joints
Links:
- removed link Link_Shoulder_le
- added link Link_Shoulder_rf, mass 0.09598; collision mesh filename=package://chyPapa5/meshes/Link_Shoulder_rf.STL; visual mesh filename=package://chyPapa5/meshes/Link_Shoulder_rf.STL
- link base_link: mass 0.302284486397825 -> 0.30153
Joints:
- removed joint Joint_Shoulder_le
- added joint Joint_Shoulder_rf: type revolute, parent base_link, child Link_Shoulder_rf, origin xyz=0.0685 -0.019304 -0.034561 rpy=-1.5708 0.034331 -1.5708, axis 0 0 -1, limit lower=1.5 upper=0.5 effort=100 velocity=0

Commit message: DH2

File: urdf/chyPapa5/urdf/chyPapa5.urdf (robot description, URDF)
Before this commit: robot chyPapa5, 2 links, 1 joints
Joints:
- joint Joint_Shoulder_rf: axis 0 0 -1 -> 0 1 0; origin xyz=0.0685 -0.019304 -0.034561 rpy=-1.5708 0.034331 -1.5708 -> xyz=0.034561 0.0685 0.019304 rpy=0 0.034331 0

Commit message: DH3

File: urdf/chyPapa5/urdf/chyPapa5.urdf (robot description, URDF)
Before this commit: robot chyPapa5, 2 links, 1 joints
Links:
- removed link Link_Shoulder_rf
- added link Link_Shoulder_Rf, mass 0.09598; collision mesh filename=package://chyPapa5/meshes/Link_Shoulder_Rf.STL; visual mesh filename=package://chyPapa5/meshes/Link_Shoulder_Rf.STL
Joints:
- removed joint Joint_Shoulder_rf
- added joint Joint_Shoulder_Rf: type revolute, parent base_link, child Link_Shoulder_Rf, origin xyz=0.0725 -0.019304 -0.034561 rpy=3.1416 -1.5708 0, axis 0 0 1, limit lower=1.5 upper=0.5 effort=100 velocity=0

Commit message: dh4

File: urdf/chyPapa5/urdf/chyPapa5.urdf (robot description, URDF)
Before this commit: robot chyPapa5, 2 links, 1 joints
Joints:
- joint Joint_Shoulder_Rf: origin xyz=0.0725 -0.019304 -0.034561 rpy=3.1416 -1.5708 0 -> xyz=0.0725 -0.034561 0.014304 rpy=-1.5708 0 1.5708

Commit message: dh3

File: urdf/chyPapa5/urdf/chyPapa5.urdf (robot description, URDF)
Before this commit: robot chyPapa5, 2 links, 1 joints
Links:
- removed link Link_Shoulder_Rf
- added link Link_Shoulder_rf, mass 0.09598; collision mesh filename=package://chyPapa5/meshes/Link_Shoulder_rf.STL; visual mesh filename=package://chyPapa5/meshes/Link_Shoulder_rf.STL
- link base_link: mass 0.30153 -> 0.301530504160963
Joints:
- removed joint Joint_Shoulder_Rf
- added joint Joint_Shoulder_rf: type revolute, parent base_link, child Link_Shoulder_rf, origin xyz=0.0725 0.019059 0.035943 rpy=3.1416 1.5708 0, axis 0 0 1, limit lower=0.5 upper=1.5 effort=0 velocity=0

Commit message: dh3

File: urdf/chyPapa5/urdf/chyPapa5.urdf (robot description, URDF)
Before this commit: robot chyPapa5, 2 links, 1 joints
Joints:
- joint Joint_Shoulder_rf: axis 0 0 1 -> 0 0 -1; limit lower=0.5 upper=1.5 effort=0 velocity=0 -> lower=0.5 upper=1.5 effort=100 velocity=0; origin xyz=0.0725 0.019059 0.035943 rpy=3.1416 1.5708 0 -> xyz=0.0685 0.019059 0.035943 rpy=-1.5708 1.49 -1.5708

Commit message: dh3

File: urdf/chyPapa5/urdf/chyPapa5.urdf (robot description, URDF)
Before this commit: robot chyPapa5, 2 links, 1 joints
Links:
- removed link Link_Shoulder_rf
- added link link_shoulder_rf, mass 0.09598; collision mesh filename=package://chyPapa5/meshes/link_shoulder_rf.STL; visual mesh filename=package://chyPapa5/meshes/link_shoulder_rf.STL
Joints:
- removed joint Joint_Shoulder_rf
- added joint joint_shoulder_rf: type revolute, parent base_link, child link_shoulder_rf, origin xyz=0.0685 0.019059 0.035943 rpy=-1.5708 1.49 -1.5708, axis 0 0 -1, limit lower=1.5 upper=0.5 effort=100 velocity=0

Commit message: chyPapa02

File: urdf/chyPapa5/urdf/chyPapa5.urdf (robot description, URDF)
Before this commit: robot chyPapa5, 2 links, 1 joints
Links:
- removed link link_shoulder_rf
- added link Link_Arm_Motor_le, mass 0.0341422557519; collision mesh filename=package://chyPapa5/meshes/Link_Arm_Motor_le.STL; visual mesh filename=package://chyPapa5/meshes/Link_Arm_Motor_le.STL
- added link Link_Arm_Motor_lf, mass 0.0341422557519; collision mesh filename=package://chyPapa5/meshes/Link_Arm_Motor_lf.STL; visual mesh filename=package://chyPapa5/meshes/Link_Arm_Motor_lf.STL
- added link Link_Arm_Motor_re, mass 0.0341422557519; collision mesh filename=package://chyPapa5/meshes/Link_Arm_Motor_re.STL; visual mesh filename=package://chyPapa5/meshes/Link_Arm_Motor_re.STL
- added link Link_Arm_Motor_rf, mass 0.0341422557519; collision mesh filename=package://chyPapa5/meshes/Link_Arm_Motor_rf.STL; visual mesh filename=package://chyPapa5/meshes/Link_Arm_Motor_rf.STL
- added link Link_Arm_le, mass 0.108265195096751; collision mesh filename=package://chyPapa5/meshes/Link_Arm_le.STL; visual mesh filename=package://chyPapa5/meshes/Link_Arm_le.STL
- added link Link_Arm_lf, mass 0.108265195096751; collision mesh filename=package://chyPapa5/meshes/Link_Arm_lf.STL; visual mesh filename=package://chyPapa5/meshes/Link_Arm_lf.STL
- added link Link_Arm_re, mass 0.108265195096751; collision mesh filename=package://chyPapa5/meshes/Link_Arm_re.STL; visual mesh filename=package://chyPapa5/meshes/Link_Arm_re.STL
- added link Link_Arm_rf, mass 0.108265195096751; collision mesh filename=package://chyPapa5/meshes/Link_Arm_rf.STL; visual mesh filename=package://chyPapa5/meshes/Link_Arm_rf.STL
- added link Link_Hand_le, mass 0.0420735853495988; collision mesh filename=package://chyPapa5/meshes/Link_Hand_le.STL; visual mesh filename=package://chyPapa5/meshes/Link_Hand_le.STL
- added link Link_Hand_lf, mass 0.0420735853495988; collision mesh filename=package://chyPapa5/meshes/Link_Hand_lf.STL; visual mesh filename=package://chyPapa5/meshes/Link_Hand_lf.STL
- added link Link_Hand_re, mass 0.0420735853495988; collision mesh filename=package://chyPapa5/meshes/Link_Hand_re.STL; visual mesh filename=package://chyPapa5/meshes/Link_Hand_re.STL
- added link Link_Hand_rf, mass 0.0420735853495988; collision mesh filename=package://chyPapa5/meshes/Link_Hand_rf.STL; visual mesh filename=package://chyPapa5/meshes/Link_Hand_rf.STL
- added link Link_Shoulder_Arm_Motor_le, mass 0.0341422557519; collision mesh filename=package://chyPapa5/meshes/Link_Shoulder_Arm_Motor_le.STL; visual mesh filename=package://chyPapa5/meshes/Link_Shoulder_Arm_Motor_le.STL
- added link Link_Shoulder_Arm_Motor_lf, mass 0.0341422557519; collision mesh filename=package://chyPapa5/meshes/Link_Shoulder_Arm_Motor_lf.STL; visual mesh filename=package://chyPapa5/meshes/Link_Shoulder_Arm_Motor_lf.STL
- added link Link_Shoulder_Arm_Motor_re, mass 0.0341422557519; collision mesh filename=package://chyPapa5/meshes/Link_Shoulder_Arm_Motor_re.STL; visual mesh filename=package://chyPapa5/meshes/Link_Shoulder_Arm_Motor_re.STL
- added link Link_Shoulder_Arm_Motor_rf, mass 0.0341422557519; collision mesh filename=package://chyPapa5/meshes/Link_Shoulder_Arm_Motor_rf.STL; visual mesh filename=package://chyPapa5/meshes/Link_Shoulder_Arm_Motor_rf.STL
- added link Link_Shoulder_Motor_le, mass 0.0341422557519; collision mesh filename=package://chyPapa5/meshes/Link_Shoulder_Motor_le.STL; visual mesh filename=package://chyPapa5/meshes/Link_Shoulder_Motor_le.STL
- added link Link_Shoulder_Motor_lf, mass 0.0341422557519; collision mesh filename=package://chyPapa5/meshes/Link_Shoulder_Motor_lf.STL; visual mesh filename=package://chyPapa5/meshes/Link_Shoulder_Motor_lf.STL
- added link Link_Shoulder_Motor_re, mass 0.0341422557519; collision mesh filename=package://chyPapa5/meshes/Link_Shoulder_Motor_re.STL; visual mesh filename=package://chyPapa5/meshes/Link_Shoulder_Motor_re.STL
- added link Link_Shoulder_Motor_rf, mass 0.0341422557519; collision mesh filename=package://chyPapa5/meshes/Link_Shoulder_Motor_rf.STL; visual mesh filename=package://chyPapa5/meshes/Link_Shoulder_Motor_rf.STL
- added link Link_Shoulder_Sheft_le, mass 0.027695; collision mesh filename=package://chyPapa5/meshes/Link_Shoulder_Sheft_le.STL; visual mesh filename=package://chyPapa5/meshes/Link_Shoulder_Sheft_le.STL
- added link Link_Shoulder_Sheft_lf, mass 0.02712; collision mesh filename=package://chyPapa5/meshes/Link_Shoulder_Sheft_lf.STL; visual mesh filename=package://chyPapa5/meshes/Link_Shoulder_Sheft_lf.STL
- added link Link_Shoulder_Sheft_re, mass 0.02712; collision mesh filename=package://chyPapa5/meshes/Link_Shoulder_Sheft_re.STL; visual mesh filename=package://chyPapa5/meshes/Link_Shoulder_Sheft_re.STL
- added link Link_Shoulder_Sheft_rf, mass 0.027695; collision mesh filename=package://chyPapa5/meshes/Link_Shoulder_Sheft_rf.STL; visual mesh filename=package://chyPapa5/meshes/Link_Shoulder_Sheft_rf.STL
Joints:
- removed joint joint_shoulder_rf
- added joint Joint_Arm_Motor_le: type fixed, parent Link_Arm_le, child Link_Arm_Motor_le, origin xyz=0 -0.13 -0.021 rpy=-3.1416 0 0, axis 0 0 0
- added joint Joint_Arm_Motor_lf: type fixed, parent Link_Arm_lf, child Link_Arm_Motor_lf, origin xyz=-0.00011618 -0.13 -0.021 rpy=-3.1416 0 0, axis 0 0 0
- added joint Joint_Arm_Motor_re: type fixed, parent Link_Arm_re, child Link_Arm_Motor_re, origin xyz=-0.00011618 -0.13 -0.021 rpy=-3.1416 0 0, axis 0 0 0
- added joint Joint_Arm_Motor_rf: type fixed, parent Link_Arm_rf, child Link_Arm_Motor_rf, origin xyz=0 0 0 rpy=0 0 0, axis 0 0 0
- added joint Joint_Arm_le: type revolute, parent Link_Shoulder_Arm_Motor_le, child Link_Arm_le, origin xyz=0 0 -0.004 rpy=-3.1416 0 -1.7063, axis 0 0 1, limit lower=-1.5 upper=1.5 effort=100 velocity=0
- added joint Joint_Arm_lf: type revolute, parent Link_Shoulder_Arm_Motor_lf, child Link_Arm_lf, origin xyz=0.0014362 0 -0.14552 rpy=-0.018505 0.0020175 1.6794, axis 0 0 1, limit lower=-1.5 upper=1.5 effort=100 velocity=0
- added joint Joint_Arm_re: type revolute, parent Link_Shoulder_Arm_Motor_re, child Link_Arm_re, origin xyz=0 0 -0.004 rpy=-3.1416 0 1.4248, axis 0 0 1, limit lower=-1.5 upper=1.5 effort=100 velocity=0
- added joint Joint_Arm_rf: type revolute, parent Link_Shoulder_Arm_Motor_rf, child Link_Arm_rf, origin xyz=0 0 -0.004 rpy=-3.1416 0 -1.4956, axis 0 0 -1, limit lower=-1.5 upper=1.5 effort=100 velocity=0
- added joint Joint_Hand_le: type revolute, parent Link_Arm_Motor_le, child Link_Hand_le, origin xyz=0 0 -0.00400000000000014 rpy=3.14159265358979 0 0.346767054762826, axis 0 0 -1, limit lower=-1.5 upper=1.5 effort=100 velocity=0
- added joint Joint_Hand_lf: type revolute, parent Link_Arm_Motor_lf, child Link_Hand_lf, origin xyz=0 0 -0.004 rpy=3.1416 0 0.060606, axis 0 0 -1, limit lower=-1.5 upper=1.5 effort=100 velocity=0
- added joint Joint_Hand_re: type revolute, parent Link_Arm_Motor_re, child Link_Hand_re, origin xyz=0 0 -0.004 rpy=3.1416 0 0.027556, axis 0 0 -1, limit lower=-1.5 upper=1.5 effort=100 velocity=0
- added joint Joint_Hand_rf: type revolute, parent Link_Arm_Motor_rf, child Link_Hand_rf, origin xyz=-0.0001166 -0.13 -0.017 rpy=0 0 0.1987, axis 0 0 -1, limit lower=-1.5 upper=1.5 effort=100 velocity=0
- added joint Joint_Shoulder_Arm_Motor_le: type fixed, parent Link_Shoulder_Sheft_le, child Link_Shoulder_Arm_Motor_le, origin xyz=-0.011 -0.027961 0.015072 rpy=0 -1.5682 1.5708, axis 0 0 0
- added joint Joint_Shoulder_Arm_Motor_lf: type fixed, parent Link_Shoulder_Sheft_lf, child Link_Shoulder_Arm_Motor_lf, origin xyz=0.011 0.12153 0.016273 rpy=0 -1.5522 -1.5708, axis 0 0 0
- added joint Joint_Shoulder_Arm_Motor_re: type fixed, parent Link_Shoulder_Sheft_re, child Link_Shoulder_Arm_Motor_re, origin xyz=-0.0279999999999998 0.014 -0.0150000000000001 rpy=3.14159265358979 -1.5707963267949 0, axis 0 0 0
- added joint Joint_Shoulder_Arm_Motor_rf: type fixed, parent Link_Shoulder_Sheft_rf, child Link_Shoulder_Arm_Motor_rf, origin xyz=0.011 0.027825 0.015322 rpy=0 -1.5593 -1.5708, axis 0 0 0
- added joint Joint_Shoulder_Motor_le: type revolute, parent base_link, child Link_Shoulder_Motor_le, origin xyz=-0.0685 0.034561 0.019304 rpy=1.5708 -1.5682 1.5708, axis 0 0 1, limit lower=-0.5 upper=1.5 effort=100 velocity=0
- added joint Joint_Shoulder_Motor_lf: type revolute, parent base_link, child Link_Shoulder_Motor_lf, origin xyz=0.0685 0.033057 0.019066 rpy=1.5708 1.5637 -1.5708, axis 0 0 1, limit lower=-0.5 upper=1.5 effort=100 velocity=0
- added joint Joint_Shoulder_Motor_re: type revolute, parent base_link, child Link_Shoulder_Motor_re, origin xyz=-0.0685 -0.034439 0.019349 rpy=1.5708 1.5659 1.5708, axis 0 0 1, limit lower=-0.5 upper=1.5 effort=100 velocity=0
- added joint Joint_Shoulder_Motor_rf: type revolute, parent base_link, child Link_Shoulder_Motor_rf, origin xyz=0.0685 -0.035943 0.019059 rpy=1.5708 -1.5593 -1.5708, axis 0 0 1, limit lower=-0.5 upper=1.5 effort=100 velocity=0
- added joint Joint_Shoulder_Sheft_le: type fixed, parent Link_Shoulder_Motor_le, child Link_Shoulder_Sheft_le, origin xyz=-0.01 -0.011 -0.028 rpy=3.139 -1.5708 0, axis 0 0 0
- added joint Joint_Shoulder_Sheft_lf: type fixed, parent Link_Shoulder_Motor_lf, child Link_Shoulder_Sheft_lf, origin xyz=0.01 -0.011 -0.028 rpy=0 1.5708 0, axis 0 0 0
- added joint Joint_Shoulder_Sheft_re: type fixed, parent Link_Shoulder_Motor_re, child Link_Shoulder_Sheft_re, origin xyz=0.01 -0.011 -0.028 rpy=-1.5708 0 1.5708, axis 0 0 0
- added joint Joint_Shoulder_Sheft_rf: type fixed, parent Link_Shoulder_Motor_rf, child Link_Shoulder_Sheft_rf, origin xyz=-0.00999999999999998 -0.0140000000000001 -0.028 rpy=3.13005288457324 1.5707963267949 0, axis 0 0 0
